File: Recovery.kicad_sch (KiCad schematic)
At the start: 37 parts, among them J1 DE9_Plug, J2 SWD Header, J3 JST-GH, J4 SWD Header, J5 JST-GH, J6 Micro-Fit, SW1 EVQ-PUC02K, U1 STM32F042F6P6TR, U2 AZ1117I-3.3, U3 L7805, U4 MCP2562-E-SN, Y1 8M, ?p

Commit message: organise schematic into sections
Parts:
- removed J2: SWD Header, Connector_PinHeader_2.54mm:PinHeader_1x04_P2.54mm_Vertical, symbol Connector_Generic:Conn_01x04
- removed J5: JST-GH, Connector_JST:JST_GH_SM04B-GHS-TB_1x04-1MP_P1.25mm_Horizontal, symbol Connector_Generic_MountingPin:Conn_01x04_MountingPin
- added J7: Micro-Fit, Connector_Molex:Molex_Micro-Fit_3.0_43045-0400_2x02_P3.00mm_Horizontal, symbol Connector_Generic:Conn_01x04
Connections:
- net +3.3V: now also J7.1 (Pin_1)
- net DEPLOYMENT_SIGNAL: now also J7.3 (Pin_3)
- net GND: now also J7.4 (Pin_4)
- net SERVO_FEEDBACK: now also J7.2 (Pin_2)
Other:
- note added: "3V3 Voltage Regulators"
- note added: "5V Voltage Regulators"
- note added: "Battery connector"
- note added: "CAN Bus connector"
- note added: "CAN Bus controller"
- note added: "Clock"
- note added: "D-Sub connector"
- note added: "Microcontroller"
- note added: "Mounting Holes"
- note added: "SW connector"
- note added: "Servo Connector"
- note removed: "is this the right connector/number of leads ?"
- note removed: "no frequency change for clock?"
- note removed: "st-link?"
- moved on the sheet: C1, C10, C11, C12, C13, C14, C2, C3, C4, C5, C6, C7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

Commit message: update pcb and schematic
Parts:
- removed H3, H4: MountingHole_Pad, MountingHole:MountingHole_3.2mm_M3_Pad_Via, symbol Mechanical:MountingHole_Pad
- removed J7: Micro-Fit, Connector_Molex:Molex_Micro-Fit_3.0_43045-0400_2x02_P3.00mm_Horizontal, symbol Connector_Generic:Conn_01x04
- removed SW1: EVQ-PUC02K, Button_Switch_SMD:Panasonic_EVQPUL_EVQPUC, symbol Switch:SW_SPST
- added C15, C16: 100n, Capacitor_SMD:C_0603_1608Metric, symbol Device:C_Small
- added J2, J5: JST-GH, Connector_JST:JST_GH_SM04B-GHS-TB_1x04-1MP_P1.25mm_Horizontal, symbol Connector_Generic_MountingPin:Conn_01x04_MountingPin
- added J8: Micro-Fit, Connector_Molex:Molex_Micro-Fit_3.0_43045-0412_2x02_P3.00mm_Vertical, symbol Connector_Generic:Conn_01x04
- added R1: 10K, Resistor_SMD:R_0603_1608Metric, symbol Device:R_Small
- added TH1: Thermistor_NTC, Resistor_SMD:R_0603_1608Metric, symbol Device:Thermistor_NTC
- added U5, U6, U8: INA350ABSIDSGR, WSON8_DSG_TEX, symbol 2023-07-04_13-01-56:INA350ABSIDSGR
- H1, H2: footprint MountingHole:MountingHole_3.2mm_M3_Pad_Via -> MountingHole:MountingHole_2.2mm_M2
- J1: footprint (none) -> Connector_Dsub:DSUB-9_Female_Vertical_P2.77x2.84mm_MountingHoles
- J6: footprint Connector_Molex:Molex_Micro-Fit_3.0_43045-0400_2x02_P3.00mm_Horizontal -> Connector_Molex:Molex_Micro-Fit_3.0_43045-0412_2x02_P3.00mm_Vertical
Connections:
- net +3.3V is gone; now on net +3V3: U1.16 (VDD)
- net +3V3: now also J4.4 (Pin_4), J2.4 (Pin_4), J5.4 (Pin_4), J8.4 (Pin_4), R1.2, U5.7 (V+), U6.7 (V+), U8.7 (V+); no longer J4.1 (Pin_1)
- net +BATT: now also J1.9; no longer J1.5
- net +VDC: now also J1.8; no longer J1.9
- net CAN+: now also J1.7; no longer J1.2
- net CAN-: now also J1.2; no longer J1.6
- net DEPLOYMENT_SIGNAL: now also J1.1, J8.3 (Pin_3); no longer J1.4
- net GND: now also J1.3, J1.5, J1.6, J3.1 (Pin_1), J4.1 (Pin_1), C15.1, C16.1, J2.1 (Pin_1), J2.MP (MountPin), J5.1 (Pin_1), J5.MP (MountPin), J8.1 (Pin_1), TH1.2, U5.4 (V-), U5.5 (REF), U6.2 (IN-), U6.4 (V-), U6.5 (REF), U8.4 (V-), U8.5 (REF); no longer J1.1, J1.7, J1.8, J3.4 (Pin_4), J4.4 (Pin_4)
- net PRESSURE_SENSOR_1: now also U1.13 (PA7), U6.6 (OUT); no longer U1.12 (PA6)
- net PRESSURE_SENSOR_2: now also U1.12 (PA6), U8.6 (OUT); no longer U1.13 (PA7)
- net SERVO_FEEDBACK: now also J8.2 (Pin_2)
- net at F1.1: now also J3.4 (Pin_4); no longer J3.1 (Pin_1)
- net TEMPERATURE_SENSOR: now reaches U1.10 (PA4)
- net TEMPERATURE_SENSOR: now also R1.1, TH1.1
- net NRST: no longer names the net of C9.2
- net NRST: no longer U1.4 (NRST)
- new net: J5.2 (Pin_2), U8.2 (IN-)
- new net: J5.3 (Pin_3), U8.3 (IN+)
- new net: U5.6 (OUT), U6.3 (IN+)
- new net: J2.2 (Pin_2), U5.2 (IN-)
- new net: J2.3 (Pin_3), U5.3 (IN+)
- no-connect marks 1 -> 16
Other:
- note added: "Gain Selection high or no connect = Gain of 20"
- note added: "Pressure Sensor 1 20*20=400 Gain"
- note added: "Pressure Sensor 2 20 Gain"
- note added: "SHDN high or no connect = device enabled"
- note added: "Temperature Sensor"
- note added: "another d sub?"
- note added: "for firmware flashing and debugging"
- note added: "high voltage protection? 9v"
- note added: "voltage divider"
- moved on the sheet: C12, C14, J1, J4, J6

Commit message: fix pcb size
Parts:
- removed C15, C16, C9: 100n, Capacitor_SMD:C_0603_1608Metric, symbol Device:C_Small
- added R2: 1K8, Resistor_SMD:R_0603_1608Metric, symbol Device:R_Small
- added R3: 1K, Resistor_SMD:R_0603_1608Metric, symbol Device:R_Small
- J2, J3, J5: footprint Connector_JST:JST_GH_SM04B-GHS-TB_1x04-1MP_P1.25mm_Horizontal -> Connector_JST:JST_GH_BM04B-GHS-TBT_1x04-1MP_P1.25mm_Vertical
Connections:
- net DEPLOYMENT_SIGNAL: now also R2.2; no longer U1.9 (PA3)
- net GND: now also R3.1; no longer H1.1, H2.1
- net at U8.2 (IN-): now also J5.3 (Pin_3); no longer J5.2 (Pin_2)
- net at U8.3 (IN+): now also J5.2 (Pin_2); no longer J5.3 (Pin_3)
- net at J2.2 (Pin_2): now also U5.3 (IN+); no longer U5.2 (IN-)
- net at J2.3 (Pin_3): now also U5.2 (IN-); no longer U5.3 (IN+)
- new net DEPLOYMENT_PIN: R2.1, R3.2, U1.9 (PA3)
- no-connect marks 16 -> 18
Other:
- note removed: "high voltage protection? 9v"
- note removed: "voltage divider"

Commit message: finish traces
Parts:
- removed H2: MountingHole_Pad, MountingHole:MountingHole_2.2mm_M2, symbol Mechanical:MountingHole_Pad
Connections:
- no-connect marks 18 -> 17
Changed lines of the file:
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@@
   (no_connect (at 234.95 248.92))
   (no_connect (at 262.89 181.61))
-  (no_connect (at 40.64 35.56))
   (no_connect (at 222.25 179.07))
   (no_connect (at 194.31 246.38))
@@
         )
       )
-    )
-  )
-  (symbol (lib_id "Mechanical:MountingHole_Pad") (at 43.18 35.56 270) (unit 1)
-    (in_bom no) (on_board yes) (dnp no)
-    (property "Reference" "H2" (at 46.99 35.56 90)
-      (effects (font (size 1.27 1.27)) (justify left))
-    )
-    (property "Value" "MountingHole_Pad" (at 46.99 37.2622 90)
-      (effects (font (size 1.27 1.27)) (justify left) hide)
-    )
-    (property "Footprint" "MountingHole:MountingHole_2.2mm_M2" (at 43.18 35.56 0)
-      (effects (font (size 1.27 1.27)) hide)
-    )
-    (property "Datasheet" "~" (at 43.18 35.56 0)
-      (effects (font (size 1.27 1.27)) hide)
-    )
-    (property "Manufacturer" "N/A" (at 43.18 35.56 0)
-      (effects (font (size 1.27 1.27)) hide)
-    )
-    (property "Part#" "N/A" (at 43.18 35.56 0)
-      (effects (font (size 1.27 1.27)) hide)
-    )
-    (property "DigiKey#" "N/A" (at 43.18 35.56 0)
-      (effects (font (size 1.27 1.27)) hide)
-    )
-    (property "LCSC#" "N/A" (at 43.18 35.56 0)
-      (effects (font (size 1.27 1.27)) hide)
-    )
-    (pin "1")
-    (instances
-      (project "Recovery"
-        (path "/1e2fd741-2f4a-40f4-b342-72b7a5b02b38"
-          (reference "H2") (unit 1)
-        )
-      )
-      (project "euroc_fc"
-        (path "/e63e39d7-6ac0-4ffd-8aa3-1841a4541b55"
-          (reference "H1") (unit 1)
-        )
-      )

Commit message: Various small fixes
- increased trace width for deploy signal, removed thermal relief
- left some room around screw, used pad hole type
- tweaked CAN traces
- Added bypass caps to amps, CAN controller
- Removed 5V rail diode & LED, diode used for BAT instead
- Used male D-Sub footprint instead of female (affects pin numbering)
- Added test points for amps
- Pulled BOOT pin low w/ 10k
- Added a jumper to allow differentiating between top and bottom
  recovery
- Add two MCU controllable LEDs
- Added silkscreen (name, rev, logo)
- Added oscillator values
- Added a voltage-divider jumper for one sensor input
- Finished BOM
Parts:
- removed D2: ~, Diode_SMD:D_SOD-123F, symbol Device:D_Schottky_Small
- added C15, C16, C17, C18, C9: 100n, Capacitor_SMD:C_0603_1608Metric, symbol Device:C_Small
- added D1: ~, Diode_SMD:D_SOD-123F, symbol Device:D_Schottky_Small
- added D2: green, LED_SMD:LED_0603_1608Metric, symbol Device:LED_Small
- added JP1: SolderJumper_2_Open, Jumper:SolderJumper-2_P1.3mm_Open_RoundedPad1.0x1.5mm, symbol Jumper:SolderJumper_2_Open
- added R10, R9: DNP, Resistor_SMD:R_0603_1608Metric, symbol Device:R_Small
- added R4: 10k, Resistor_SMD:R_0603_1608Metric, symbol Device:R_Small
- added R8: 1k, Resistor_SMD:R_0603_1608Metric, symbol Device:R_Small
- added TP1, TP2, TP3, TP4, TP5, TP6, TP7: TestPoint, TestPoint:TestPoint_Pad_D2.0mm, symbol Connector:TestPoint
- C1, C2: value 22p -> 10p; LCSC# C1653 -> C1634; Part# CL10C220JB8NNNC -> CL10C100JB8NNNC
- H1: footprint MountingHole:MountingHole_2.2mm_M2 -> MountingHole:MountingHole_2.2mm_M2_Pad
- J1: footprint Connector_Dsub:DSUB-9_Female_Vertical_P2.77x2.84mm_MountingHoles -> Connector_Dsub:DSUB-9_Male_Vertical_P2.77x2.84mm_MountingHoles; DigiKey# (none) -> 609-5545-ND; Manufacturer (none) -> Amphenol ICC (FCI); Part# (none) -> D09P24A4PL00LF
- J2, J3, J5: LCSC# C189895 -> C161692; Part# SM04B-GHS-TB -> BM04B-GHS-TBT
- J4: DigiKey# (none) -> N/A; LCSC# (none) -> N/A; Manufacturer (none) -> N/A; Part# (none) -> N/A
- J6, J8: DigiKey# (none) -> WM1790-ND; LCSC# C122413 -> (none); Part# 0430450400 -> 0430450412
- R1: value 10K -> 10k; LCSC# C105881 -> C98220; Part# RC0603FR-07330RL -> RC0603FR-0710KL
- R2: value 1K8 -> 1k8; LCSC# C105881 -> C185354; Part# RC0603FR-07330RL -> RC0603FR-071K8L
- R3: value 1K -> 1k; LCSC# C105881 -> C22548; Part# RC0603FR-07330RL -> RC0603FR-071KL
- R5: value 330 -> 1k; LCSC# C105881 -> C22548; Part# RC0603FR-07330RL -> RC0603FR-071KL
- R6: value 220 -> 1k; LCSC# C2085669 -> C22548; Manufacturer ROHM Semicon -> YAGEO; Part# ESR03EZPJ221 -> RC0603FR-071KL
- TH1: value Thermistor_NTC -> NCU18XH103F6SRB; DigiKey# (none) -> 490-18139-1-ND; Manufacturer (none) -> Murata Electronics; Part# (none) -> NCU18XH103F6SRB
- U1: DigiKey# (none) -> 497-19656-1-ND; Manufacturer (none) -> STMicroelectronics; Part# (none) -> STM32F042F6P6TR
- U5, U6: footprint WSON8_DSG_TEX -> footprints2:WSON8_DSG_TEX; DigiKey# (none) -> 296-INA350ABSIDSGRCT-ND; Manufacturer (none) -> Texas Instruments; Part# (none) -> INA350ABSIDSGR
- U7: renamed from U8; footprint WSON8_DSG_TEX -> footprints2:WSON8_DSG_TEX; DigiKey# (none) -> 296-INA350ABSIDSGRCT-ND; Manufacturer (none) -> Texas Instruments; Part# (none) -> INA350ABSIDSGR
- Y1: value 8M, ?p -> 8M, 12p; DigiKey# (none) -> 50-ECS-80-12-33-JGN-CT-ND; LCSC# C255956 -> (none); Manufacturer Seiko Epson -> ECS Inc.; Part# Q24FA20H0039000 -> ECS-80-12-33-JGN-TR
Connections:
- net +3V3: now also D3.2 (A), C16.2, C17.2, C18.2, C9.2, D2.2 (A)
- net +5V: now also C11.2, U3.3 (OUT), C15.2
- net +BATT: now also D1.2 (A); no longer C5.2, U3.1 (IN)
- net GND: now also H1.1, C15.1, C16.1, C17.1, C18.1, C9.1, JP1.1 (A), R10.1, R4.1; no longer D3.1 (K)
- net PRESSURE_SENSOR_1: now also TP4.1
- net PRESSURE_SENSOR_2: now also R10.2, R9.1, TP7.1
- net SERVO_FEEDBACK: now also U1.8 (PA2); no longer U1.7 (PA1)
- net LED_GREEN: now reaches R6.2
- net LED_GREEN: now also U1.7 (PA1); no longer D3.2 (A)
- net at J5.3 (Pin_3), U7.2 (IN-): now also TP5.1
- net at J5.2 (Pin_2), U7.3 (IN+): now also R9.2, TP6.1
- net at U5.6 (OUT), U6.3 (IN+): now also TP3.1
- net at J2.2 (Pin_2), U5.3 (IN+): now also TP2.1
- net at J2.3 (Pin_3), U5.2 (IN-): now also TP1.1
- net BOOT: now reaches U1.1 (PB8)
- net BOOT: now also R4.2
- net ADDRESS: now reaches U1.11 (PA5)
- net ADDRESS: now also JP1.2 (B)
- net LED_RED: now reaches U1.6 (PA0)
- net LED_RED: now also R8.2
- new net: D3.1 (K), R8.1
- new net: D2.1 (K), R6.1
- new net: C5.2, D1.1 (K), U3.1 (IN)
- no-connect marks 17 -> 12
Other:
- moved on the sheet: C11, C5, R2, R3, R7, U3, U4
